Commit message: initial gripper work commit

File: husky_description/urdf/description.xacro (robot description, xacro)
@@ -25,4 +25,5 @@
   <xacro:arg name="ur5_enabled" default="false" />
   <xacro:arg name="kinect_enabled" default="false" />
+  <xacro:arg name="gripper_enabled" default="false" />
   <xacro:include filename="$(find husky_description)/urdf/husky.urdf.xacro" />
   <xacro:husky_robot />

File: husky_description/urdf/husky.urdf.xacro (robot description, xacro)
@@ -29,4 +29,5 @@
   <xacro:include filename="$(find husky_description)/urdf/accessories/sensor_arch.urdf.xacro"/>
   <xacro:include filename="$(find ur_description)/urdf/ur5.urdf.xacro" />
+  <xacro:include filename="$(find pr2_description)/urdf/gripper_v0/gripper.urdf.xacro"/>
   <property name="M_PI" value="3.14159"/>
   <!-- Base Size -->
@@ -117,4 +118,19 @@
         <origin xyz="0.3058 0 0.0065" rpy="0.0 0.0 -1.57" />
       </joint>
+	      <xacro:if value="$(arg gripper_enabled)">
+		       <xacro:pr2_gripper_v0 reflect="-1.0" side="r" parent="ur5_arm_ee_link"
+			       screw_reduction="${4.0/1000.0}"
+			       gear_ratio="${(729.0/25.0)*(22.0/16.0)}"
+			       theta0="${3.6029*M_PI/180.0}"
+			       phi0="${29.7089*M_PI/180.0}"
+			       t0="${-0.1914/1000.0}"
+			       L0="${37.5528/1000.0}"
+			       h="${0.0/1000.0}"
+			       a="${68.3698/1000.0}"
+			       b="${43.3849/1000.0}"
+			       r="${91.5/1000.0}" >
+		      <origin xyz="0 0 0" rpy="0 0 0" />
+		      </xacro:pr2_gripper_v0>
+	    </xacro:if>
     </xacro:if>
     <xacro:if value="$(arg laser_enabled)">
