Commit message: Updated position of gripper

File: husky_description/urdf/husky.urdf.xacro (robot description, xacro)
@@ -130,5 +130,5 @@
 			       b="${43.3849/1000.0}"
 			       r="${91.5/1000.0}" >
-		      <origin xyz="0 0 0" rpy="0 0 0" />
+		      <origin xyz="-0.03 0 0" rpy="0 0 0" />
 		      </xacro:pr2_gripper_v0>
 	    </xacro:if>
